File: PCB/LED-Zappelin-V2-Chrolis/LED-Zappelin-V2-Chrolis.kicad_sch (KiCad schematic)
At the start: 29 parts, among them J1 Blanking Signal, J2 Trigger, J3 Chrolis 1, J4 Chrolis 2, J5 NeoPixel Strip, Q1 2N5089, Q2 2N5089, SW1 Blanking Switch, SW2 Blanking Inverter Switch, U1 ESP32-DEVKITC-32D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

Commit message: update board for chrolis
This update adds a voltage regulator to the board, as well as a connection to an external power supply. Footprints have been moved around so that only two sides of the board have connectors.
Parts:
- added J6: Barrel_Jack, Connector_BarrelJack:BarrelJack_Horizontal, symbol Connector:Barrel_Jack
- added R10: 330, Resistor_THT:R_Axial_DIN0309_L9.0mm_D3.2mm_P15.24mm_Horizontal, symbol Device:R_Small
- added R9: 1k, Resistor_THT:R_Axial_DIN0309_L9.0mm_D3.2mm_P15.24mm_Horizontal, symbol Device:R_Small
- added U5: LM317_TO-220, Package_TO_SOT_THT:TO-220-3_Vertical, symbol Regulator_Linear:LM317_TO-220
Connections:
- net 5V: now also R9.2, U5.2 (VO)
- net GNDREF: now also J6.2, R10.1
- net GPIO Input 10: now also U4.3; no longer U4.6
- net GPIO Input 9: now also U4.6; no longer U4.3
- net GPIO00: now also J3.4; no longer J3.3
- net GPIO02: now also J3.5; no longer J3.2
- net GPIO04: now also J3.3; no longer J3.4
- net GPIO15: now also J3.6; no longer J3.1
- net GPIO16: now also J3.2; no longer J3.5
- net GPIO17: now also J3.1; no longer J3.6
- new net: R10.2, R9.1, U5.1 (ADJ)
- new net +9V: J6.1, U5.3 (VI)
- no-connect marks 6 -> 19
Other:
- moved on the sheet: H1, H3, H4, J2, J5
