File: PCB/LED-Zappelin-V2-Chrolis/LED-Zappelin-V2-Chrolis.kicad_sch (KiCad schematic)
At the start: 33 parts, among them J1 Blanking Signal, J2 Trigger, J3 Chrolis 1, J4 Chrolis 2, J5 NeoPixel Strip, J6 Barrel_Jack, Q1 2N5089, Q2 2N5089, SW1 Blanking Switch, SW2 Blanking Inverter Switch, U1 ESP32-DEVKITC-32D, U2 74LS08, U3 74LS08, U4 74LS08, U5 LM317_TO-220

Commit message: Update PCB
Parts:
- removed R10: 330, Resistor_THT:R_Axial_DIN0309_L9.0mm_D3.2mm_P15.24mm_Horizontal, symbol Device:R_Small
- removed R9: 1k, Resistor_THT:R_Axial_DIN0309_L9.0mm_D3.2mm_P15.24mm_Horizontal, symbol Device:R_Small
- added C1, C3, C5: 1μF, Capacitor_THT:C_Radial_D5.0mm_H5.0mm_P2.00mm, symbol Device:C
- added C2, C4: 10nF, Capacitor_THT:C_Rect_L11.0mm_W4.2mm_P10.00mm_MKT, symbol Device:C
- added D5: Modulated, LED_THT:LED_D3.0mm, symbol Device:LED
- added D6: Not Modulated, LED_THT:LED_D3.0mm, symbol Device:LED
- added D7: Blanking 2ms, LED_THT:LED_D3.0mm, symbol Device:LED
- added D8: Blanking 1ms, LED_THT:LED_D3.0mm, symbol Device:LED
- added Q3, Q4, Q5, Q6, Q7: 2N5089, Package_TO_SOT_THT:TO-92L_Inline_Wide, symbol Transistor_BJT:2N2219
- added R10: 720Ω, Resistor_THT:R_Axial_DIN0309_L9.0mm_D3.2mm_P15.24mm_Horizontal, symbol Device:R
- added R11, R12, R14, R21: 220Ω, Resistor_THT:R_Axial_DIN0309_L9.0mm_D3.2mm_P15.24mm_Horizontal, symbol Device:R
- added R13, R15, R16, R19, R20: 10kΩ, Resistor_THT:R_Axial_DIN0309_L9.0mm_D3.2mm_P15.24mm_Horizontal, symbol Device:R
- added R17, R18: 1kΩ, Resistor_THT:R_Axial_DIN0309_L9.0mm_D3.2mm_P15.24mm_Horizontal, symbol Device:R
- added R9: 240Ω, Resistor_THT:R_Axial_DIN0309_L9.0mm_D3.2mm_P15.24mm_Horizontal, symbol Device:R
- added RV1: 2kΩ, Potentiometer_THT:Potentiometer_Vishay_43_Horizontal, symbol Device:R_Potentiometer
- added RV2: 1kΩ, Potentiometer_THT:Potentiometer_Vishay_43_Horizontal, symbol Device:R_Potentiometer
- added SW3: BlankingModulation Switch, Maxime:maxi_DPDT_Angled, symbol Switch:SW_Push_DPDT
- added SW4: Blanking Inverter Switch, Maxime:maxi_DPDT_Angled, symbol Switch:SW_Push_DPDT
- added U7: NE556, Package_DIP:DIP-12_W7.62mm_LongPads, symbol Timer:NE556
Connections:
- net 5V: now also C1.1, Q3.3 (C), Q4.3 (C), R17.2, R18.1, R9.1; no longer U1.19 (EXT_5V)
- net Blanking: no longer R1.2, R2.2
- net GNDREF: now also C1.2, C2.2, C3.1, C4.2, C5.1, D5.1 (K), D6.1 (K), D7.1 (K), D8.1 (K), Q6.1 (E), Q7.1 (E), R10.2, RV1.1, RV2.1, U7.7 (GND), U7.7 (GND)
- net at U5.1 (ADJ): now also R10.1, R9.2
- net at Q2.2 (B), R3.2, SW1.6 (C): now also Q3.2 (B)
- net BlankingModulated: now reaches SW1.2 (B)
- net BlankingModulated: now also SW3.3 (C), SW4.2 (B); no longer J1.1 (In)
- net +9V renamed +12V
- new net: C3.2, RV1.2, U7.1 (DIS), U7.2 (THR)
- new net: Q5.2 (B), R15.1
- new net: Q7.3 (C), R15.2, R18.2
- new net: Q7.2 (B), R19.1
- new net: D6.2 (A), R12.1
- new net: C2.1, U7.3 (CV)
- new net: R12.2, SW3.6 (C)
- new net: Q4.1 (E), SW4.5 (B)
- new net: Q4.2 (B), R11.2, SW3.4 (A)
- new net: C5.2, RV2.2, U7.12 (THR), U7.13 (DIS)
- new net: D5.2 (A), R11.1
- new net: Q3.1 (E), SW3.5 (B)
- new net: D8.2 (A), R21.1
- new net: D7.2 (A), R14.1
- new net: C4.1, U7.11 (CV)
- new net: R14.2, SW4.4 (A)
- new net: Q5.1 (E), Q6.3 (C)
- new net: Q6.2 (B), R16.1
- new net: R21.2, SW4.6 (C)
- new net BlankingModulated_1ms: SW4.3 (C), U7.9 (Q)
- new net BlankingModulated_2ms: SW4.1 (A), U7.5 (Q)
- new net BlankingSignal: J1.1 (In), R1.2, R2.2, SW3.2 (B)
- new net BlankingToModulate: R16.2, R19.2, SW3.1 (A)
- new net BlankingTrigger: Q5.3 (C), R13.1, R13.2, R17.1, R20.1, R20.2, RV1.3, RV2.3, U7.10 (R), U7.14 (VCC), U7.14 (VCC), U7.4 (R), U7.6 (TR), U7.8 (TR)
Other:
- moved on the sheet: D1, D2, D3, D4, H1, H2, H3, H4, J1, J2, J3, J4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
