File: PCB/LED-Zappelin-V2-Chrolis/LED-Zappelin-V2-Chrolis.kicad_pcb (KiCad board)
At the start: 2 copper layers, 100 x 115 mm, 34 parts, among them J1 Blanking Signal, J2 Trigger Output, J3 Chrolis 1, J4 Chrolis 2, J5 NeoPixel Strip, J6 Barrel_Jack, Q1 2N5089, Q2 2N5089, SW1 Blanking Switch, SW2 Blanking Inverter Switch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

Commit message: update PCB
Routing:
- net Blanking: track 200.7 -> 219.1 mm
- net Net-(Q2-B): track 24.4 -> 35.2 mm
- net Net-(U1-IO35): track 147.7 -> 146.9 mm
Changed lines of the file:
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@@
   (segment (start 71.34 75.2) (end 58.64 75.2) (width 0.25) (layer "F.Cu") (net 2))
   (segment (start 58.64 75.2) (end 53.1 69.66) (width 0.25) (layer "F.Cu") (net 2))
-  (segment (start 58.765 93.5) (end 75 93.5) (width 0.25) (layer "F.Cu") (net 3))
-  (segment (start 75 93.5) (end 76.6 91.9) (width 0.25) (layer "F.Cu") (net 3))
-  (segment (start 53.1 87.835) (end 58.765 93.5) (width 0.25) (layer "F.Cu") (net 3))
-  (segment (start 72.8 117.9) (end 53.135 117.9) (width 0.25) (layer "B.Cu") (net 4))
+  (segment (start 58.765 93.5) (end 75 93.5) (width 0.5) (layer "F.Cu") (net 3))
+  (segment (start 75 93.5) (end 76.6 91.9) (width 0.5) (layer "F.Cu") (net 3))
+  (segment (start 53.1 87.835) (end 58.765 93.5) (width 0.5) (layer "F.Cu") (net 3))
+  (segment (start 72.8 117.9) (end 53.135 117.9) (width 0.5) (layer "F.Cu") (net 4))
   (segment (start 53.135 117.9) (end 53.1 117.935) (width 0.25) (layer "B.Cu") (net 4))
-  (segment (start 53.1 99.635) (end 51.4 101.335) (width 0.25) (layer "B.Cu") (net 5))
-  (segment (start 51.4 112.7) (end 55.2 116.5) (width 0.25) (layer "B.Cu") (net 5))
-  (segment (start 51.4 101.335) (end 51.4 112.7) (width 0.25) (layer "B.Cu") (net 5))
-  (segment (start 75.18 116.5) (end 76.6 117.92) (width 0.25) (layer "B.Cu") (net 5))
-  (segment (start 55.2 116.5) (end 75.18 116.5) (width 0.25) (layer "B.Cu") (net 5))
+  (segment (start 55.1 101.635) (end 55.1 103.4) (width 0.5) (layer "F.Cu") (net 5))
+  (segment (start 53.2 114.5) (end 55.2 116.5) (width 0.5) (layer "F.Cu") (net 5))
+  (segment (start 75.18 116.5) (end 76.6 117.92) (width 0.5) (layer "F.Cu") (net 5))
+  (segment (start 55.2 116.5) (end 75.18 116.5) (width 0.5) (layer "F.Cu") (net 5))
+  (segment (start 55.1 103.4) (end 53.2 105.3) (width 0.5) (layer "F.Cu") (net 5))
+  (segment (start 53.2 105.3) (end 53.2 114.5) (width 0.5) (layer "F.Cu") (net 5))
+  (segment (start 53.1 99.635) (end 55.1 101.635) (width 0.5) (layer "F.Cu") (net 5))
   (segment (start 51 76.1) (end 54 79.1) (width 0.5) (layer "F.Cu") (net 6))
   (segment (start 54 79.1) (end 61.92 79.1) (width 0.5) (layer "F.Cu") (net 6))
@@
   (segment (start 136.68 92.4) (end 134 95.08) (width 0.5) (layer "F.Cu") (net 31))
   (segment (start 134 95.08) (end 134 106.44) (width 0.5) (layer "F.Cu") (net 31))
+  (segment (start 80.2 117.8) (end 80.2 53.7) (width 0.5) (layer "F.Cu") (net 32))
+  (segment (start 70.1 156.7) (end 64.2 150.8) (width 0.5) (layer "F.Cu") (net 32))
+  (segment (start 99.9 75.98) (end 108.9 84.98) (width 0.5) (layer "F.Cu") (net 32))
+  (segment (start 73.939346 120.7) (end 77.3 120.7) (width 0.5) (layer "F.Cu") (net 32))
   (segment (start 96.7 51.8) (end 99.9 55) (width 0.5) (layer "F.Cu") (net 32))
-  (segment (start 99.9 75.98) (end 108.9 84.98) (width 0.5) (layer "F.Cu") (net 32))
+  (segment (start 64.2 130.439346) (end 73.939346 120.7) (width 0.5) (layer "F.Cu") (net 32))
   (segment (start 99.9 55) (end 99.9 75.98) (width 0.5) (layer "F.Cu") (net 32))
+  (segment (start 64.2 150.8) (end 64.2 130.439346) (width 0.5) (layer "F.Cu") (net 32))
+  (segment (start 80.2 53.7) (end 82.1 51.8) (width 0.5) (layer "F.Cu") (net 32))
+  (segment (start 77.3 120.7) (end 80.2 117.8) (width 0.5) (layer "F.Cu") (net 32))
   (segment (start 82.1 51.8) (end 96.7 51.8) (width 0.5) (layer "F.Cu") (net 32))
-  (segment (start 80.2 117.525) (end 80.2 53.7) (width 0.5) (layer "F.Cu") (net 32))
-  (segment (start 78.2 119.525) (end 80.2 117.525) (width 0.5) (layer "F.Cu") (net 32))
-  (segment (start 64.2 130.439346) (end 64.2 150.8) (width 0.5) (layer "F.Cu") (net 32))
-  (segment (start 71 123.639346) (end 75.114346 119.525) (width 0.5) (layer "F.Cu") (net 32))
-  (segment (start 64.2 150.8) (end 70.1 156.7) (width 0.5) (layer "F.Cu") (net 32))
-  (segment (start 75.114346 119.525) (end 78.2 119.525) (width 0.5) (layer "F.Cu") (net 32))
-  (segment (start 71 123.639346) (end 64.2 130.439346) (width 0.5) (layer "F.Cu") (net 32))
-  (segment (start 80.2 53.7) (end 82.1 51.8) (width 0.5) (layer "F.Cu") (net 32))
   (segment (start 115 154.8) (end 113.675 156.125) (width 0.25) (layer "F.Cu") (net 34))
   (segment (start 115 154.8) (end 105.92 154.8) (width 1) (layer "B.Cu") (net 34))
   (segment (start 105.92 154.8) (end 99.12 161.6) (width 1) (layer "B.Cu") (net 34))
-  (segment (start 69 118.72) (end 62.82 112.54) (width 0.5) (layer "F.Cu") (net 35))
+  (segment (start 77.2 119.8) (end 72.8 119.8) (width 0.5) (layer "F.Cu") (net 35))
   (segment (start 103.555 123.6) (end 76.6 123.6) (width 0.5) (layer "F.Cu") (net 35))
+  (segment (start 76.44 112.54) (end 78.5 114.6) (width 0.5) (layer "F.Cu") (net 35))
   (segment (start 59.4 114.6) (end 60.76 114.6) (width 0.5) (layer "F.Cu") (net 35))
-  (segment (start 69 123.6) (end 69 118.72) (width 0.5) (layer "F.Cu") (net 35))
+  (segment (start 78.5 118.5) (end 77.2 119.8) (width 0.5) (layer "F.Cu") (net 35))
   (segment (start 57.3 112.5) (end 59.4 114.6) (width 0.5) (layer "F.Cu") (net 35))
   (segment (start 57.3 104.37) (end 57.3 112.5) (width 0.5) (layer "F.Cu") (net 35))
@@
   (segment (start 113.975 134.02) (end 103.555 123.6) (width 0.5) (layer "F.Cu") (net 35))
   (segment (start 64.77 96.9) (end 57.3 104.37) (width 0.5) (layer "F.Cu") (net 35))
+  (segment (start 72.8 119.8) (end 69 123.6) (width 0.5) (layer "F.Cu") (net 35))
+  (segment (start 62.82 112.54) (end 76.44 112.54) (width 0.5) (layer "F.Cu") (net 35))
+  (segment (start 78.5 114.6) (end 78.5 118.5) (width 0.5) (layer "F.Cu") (net 35))
   (segment (start 118.98 96.4) (end 118.98 98.94) (width 0.5) (layer "B.Cu") (net 35))
   (segment (start 121.52 104.02) (end 121.52 101.48) (width 0.5) (layer "B.Cu") (net 35))
@@
   (segment (start 74.4 100.6) (end 77.04 97.96) (width 0.5) (layer "F.Cu") (net 43))
   (segment (start 58 107.72) (end 58 106.3) (width 0.5) (layer "F.Cu") (net 43))
+  (segment (start 78.4 89.5) (end 76.2 87.3) (width 0.5) (layer "F.Cu") (net 44))
+  (segment (start 71.8 87.3) (end 72.2 87.3) (width 0.5) (layer "F.Cu") (net 44))
   (segment (start 60.28 82.54) (end 65.04 87.3) (width 0.5) (layer "F.Cu") (net 44))
   (segment (start 72.8 87.9) (end 72.8 91.9) (width 0.5) (layer "F.Cu") (net 44))
+  (segment (start 74.5 96.85) (end 78.4 92.95) (width 0.5) (layer "F.Cu") (net 44))
+  (segment (start 76.2 87.3) (end 71.8 87.3) (width 0.5) (layer "F.Cu") (net 44))
   (segment (start 72.2 87.3) (end 72.8 87.9) (width 0.5) (layer "F.Cu") (net 44))
-  (segment (start 65.04 87.3) (end 72.2 87.3) (width 0.5) (layer "F.Cu") (net 44))
-  (segment (start 74.5 93.6) (end 72.8 91.9) (width 0.5) (layer "B.Cu") (net 44))
-  (segment (start 74.5 96.85) (end 74.5 93.6) (width 0.5) (layer "B.Cu") (net 44))
+  (segment (start 78.4 92.95) (end 78.4 89.5) (width 0.5) (layer "F.Cu") (net 44))
+  (segment (start 65.04 87.3) (end 71.8 87.3) (width 0.5) (layer "F.Cu") (net 44))
+  (segment (start 80.9 118.08995) (end 80.9 53.98995) (width 0.5) (layer "F.Cu") (net 45))
+  (segment (start 80.9 53.98995) (end 82.38995 52.5) (width 0.5) (layer "F.Cu") (net 45))
+  (segment (start 99.2 77.82) (end 108.9 87.52) (width 0.5) (layer "F.Cu") (net 45))
+  (segment (start 75 122.7) (end 76.3 121.4) (width 0.5) (layer "F.Cu") (net 45))
+  (segment (start 76.3 121.4) (end 77.58995 121.4) (width 0.5) (layer "F.Cu") (net 45))
+  (segment (start 82.38995 52.5) (end 96.41005 52.5) (width 0.5) (layer "F.Cu") (net 45))
+  (segment (start 77.58995 121.4) (end 80.9 118.08995) (width 0.5) (layer "F.Cu") (net 45))
   (segment (start 96.41005 52.5) (end 99.2 55.28995) (width 0.5) (layer "F.Cu") (net 45))
-  (segment (start 99.2 77.82) (end 108.9 87.52) (width 0.5) (layer "F.Cu") (net 45))
-  (segment (start 80.9 117.81495) (end 80.9 53.98995) (width 0.5) (layer "F.Cu") (net 45))
-  (segment (start 75.675 120.225) (end 78.489949 120.225) (width 0.5) (layer "F.Cu") (net 45))
-  (segment (start 78.489949 120.225) (end 80.9 117.81495) (width 0.5) (layer "F.Cu") (net 45))
-  (segment (start 75 129.6) (end 75 120.9) (width 0.5) (layer "F.Cu") (net 45))
-  (segment (start 82.38995 52.5) (end 96.41005 52.5) (width 0.5) (layer "F.Cu") (net 45))
-  (segment (start 80.9 53.98995) (end 82.38995 52.5) (width 0.5) (layer "F.Cu") (net 45))
-  (segment (start 69 135.6) (end 75 129.6) (width 0.5) (layer "F.Cu") (net 45))
+  (segment (start 75 129.6) (end 75 122.7) (width 0.5) (layer "F.Cu") (net 45))
   (segment (start 69 138.84) (end 69 135.6) (width 0.5) (layer "F.Cu") (net 45))
   (segment (start 99.2 55.28995) (end 99.2 77.82) (width 0.5) (layer "F.Cu") (net 45))
-  (segment (start 75 120.9) (end 75.675 120.225) (width 0.5) (layer "F.Cu") (net 45))
+  (segment (start 69 135.6) (end 75 129.6) (width 0.5) (layer "F.Cu") (net 45))
   (segment (start 79.4 159.6) (end 102.2 159.6) (width 0.5) (layer "F.Cu") (net 46))
   (segment (start 77.4 157.8) (end 77.4 161.6) (width 0.5) (layer "F.Cu") (net 46))
