File: PCB/LED-Zappelin-V2-Chrolis/_autosave-LED-Zappelin-V2-Chrolis.kicad_pcb (KiCad board)
At the start: 2 copper layers, 100 x 135 mm, 68 parts, among them J1 Blanking Signal, J2 Trigger, J3 Chrolis 1, J4 Chrolis 2, J5 NeoPixel Strip, J6 Barrel_Jack, Q1 2N5089, Q2 2N5089, Q3 2N5089, Q4 2N5089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

Commit message: Update PCB
Parts:
- added J7: Power Switch, Connector_JST:JST_XH_B3B-XH-A_1x03_P2.50mm_Vertical, F.Cu at (137.3, 180.8)
- J6: value Barrel_Jack -> 12 V
- moved U5 31.1 mm to (110.4, 180.0)
Connections:
- J6 pad 1: +12V -> Net-(J7-Pin_2)
Routing:
- net +12V: track 15.2 -> 41.8 mm
- net Net-(J7-Pin_2): track 0.00 -> 15.9 mm
- net Net-(U5-ADJ): track 52.3 -> 64.6 mm
- net 5V: track 966.9 -> 959.7 mm
- net GPIO Input 1: track 38.3 -> 39.1 mm
Other:
- board text added: "- + +"
